File: DSP_MOTU1_proto.brd (EAGLE design)
At the start: 67.3 x 46.4 mm, 175 parts, among them IC1 ADAU1463WBCPZ300RL, IC2 25AA1024, IC3 ADM811TARTZ, IC4 TPS54227DDAR, IC5 WEMOS_D1_MINI, IC6 SN65MLVD205AD, J1 CON_2X18_2MM, J2 CON_2X18_2MM, Y1 ABM3B-12.288MHZ-10-1-U-T

Commit message: Add files via upload
Parts:
- moved J1 1.00 mm to (3.27, 1.50)
Routing:
- net DVDD: track 0.00 -> 62.2 mm, vias 0 -> 9
- net IOVDD: track 0.00 -> 52.8 mm, vias 0 -> 11
- net 3V3D: track 0.00 -> 50.4 mm, vias 0 -> 2
- net N$14: track 0.00 -> 35.3 mm
- net SS: track 0.00 -> 33.6 mm, vias 0 -> 2
- net MOSI: track 0.00 -> 28.8 mm, vias 0 -> 1
- net PBCKOUT0: track 0.00 -> 26.2 mm
- net SCLK: track 0.00 -> 25.8 mm, vias 0 -> 1
- net PMP7: track 0.00 -> 23.5 mm, vias 0 -> 2
- net PMP6: track 0.00 -> 23.3 mm, vias 0 -> 2
- net MP24: track 0.00 -> 22.7 mm, vias 0 -> 1
- net PMP10: track 0.00 -> 22.3 mm, vias 0 -> 4
- net DSPRST: track 0.00 -> 22.3 mm, vias 0 -> 2
- net MISO: track 0.00 -> 22.1 mm, vias 0 -> 2
- net MP25: track 0.00 -> 21.4 mm, vias 0 -> 1
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- added copper zone on layer 16, net 14V8
- added copper zone on layer 15, net DVDD
- added copper zone on layer 16, net DVDD
- added copper zone on layer 16, net GND
Other:
- board size 67.3 x 46.4 mm -> 68.3 x 46.4 mm
- board text added: "2 connectors mounted on solder side!"
- board text added: "DSP_MOTU V1 03-2019"
- board text added: "DSP_MOTU V1.0 03-2019"
- board text added: "k"
- board text removed: "MOTU_DSP8 02-2019"
- board text removed: "MOTU_DSP8 V1.0"
